Commit message: run tests for tylenol

File: src/pen_description/urdf/pen_cell.urdf.xacro (robot description, xacro)
@@ -11,4 +11,10 @@
   <xacro:arg name="profile_id" default="TBD"/>
   <xacro:arg name="surface_type" default="sphere"/>
+  <xacro:arg name="surface_radius" default="0.0291"/>
+  <xacro:arg name="surface_height" default="0.03"/>
+  <xacro:arg name="workpiece_holder_xyz" default="0 0 0"/>
+  <xacro:arg name="workpiece_holder_rpy" default="0 0 0"/>
+  <xacro:arg name="workpiece_bottle_xyz" default="0 0 0"/>
+  <xacro:arg name="workpiece_bottle_rpy" default="0 0 0"/>
   <xacro:arg name="camera_enabled" default="false"/>
   <xacro:arg name="camera_xyz" default="TBD"/><xacro:arg name="camera_rpy" default="TBD"/>

File: src/pen_description/urdf/pen_fixture.xacro (robot description, xacro)
@@ -5,4 +5,24 @@
     <joint name="base_to_pen_jig" type="fixed"><parent link="${base}"/><child link="pen_jig"/><origin xyz="${jig_xyz}" rpy="${jig_rpy}"/></joint>
     <link name="pen_surface">
+      <xacro:if value="${surface_type == 'cylinder'}">
+        <visual name="tylenol_bottle">
+          <origin xyz="$(arg workpiece_bottle_xyz)" rpy="$(arg workpiece_bottle_rpy)"/>
+          <geometry><mesh filename="package://pen_description/assets/tylenol/tylenol.glb"/></geometry>
+        </visual>
+        <visual name="tylenol_holder">
+          <origin xyz="$(arg workpiece_holder_xyz)" rpy="$(arg workpiece_holder_rpy)"/>
+          <geometry><mesh filename="package://pen_description/assets/tylenol/holder.stl"/></geometry>
+          <material name="tylenol_holder_gray"><color rgba="0.22 0.25 0.28 1"/></material>
+        </visual>
+        <collision name="bottle_proxy">
+          <origin rpy="0 1.5707963267948966 0"/>
+          <geometry><cylinder radius="$(arg surface_radius)" length="$(arg surface_height)"/></geometry>
+        </collision>
+        <collision name="holder">
+          <origin xyz="$(arg workpiece_holder_xyz)" rpy="$(arg workpiece_holder_rpy)"/>
+          <geometry><mesh filename="package://pen_description/assets/tylenol/holder.stl"/></geometry>
+        </collision>
+      </xacro:if>
+      <xacro:unless value="${surface_type == 'cylinder'}">
       <visual>
         <origin xyz="0 0 ${-0.0025 if surface_type == 'plane' else 0}"/>
@@ -13,4 +33,5 @@
         <geometry><mesh filename="package://pen_description/meshes/${'flat' if surface_type == 'plane' else 'sphere'}.stl" scale="1 1 1"/></geometry>
       </collision>
+      </xacro:unless>
     </link>
     <joint name="jig_to_pen_surface" type="fixed"><parent link="pen_jig"/><child link="pen_surface"/><origin xyz="${surface_xyz}" rpy="${surface_rpy}"/></joint>

Commit message: complete image print

File: src/pen_description/urdf/pen_cell.urdf.xacro (robot description, xacro)
@@ -13,4 +13,6 @@
   <xacro:arg name="surface_radius" default="0.0291"/>
   <xacro:arg name="surface_height" default="0.03"/>
+  <xacro:arg name="plane_visual_mesh" default=""/>
+  <xacro:arg name="plane_size_m" default="0.08 0.1 0.0025"/>
   <xacro:arg name="workpiece_holder_xyz" default="0 0 0"/>
   <xacro:arg name="workpiece_holder_rpy" default="0 0 0"/>

File: src/pen_description/urdf/pen_fixture.xacro (robot description, xacro)
@@ -25,4 +25,14 @@
       </xacro:if>
       <xacro:unless value="${surface_type == 'cylinder'}">
+      <xacro:if value="${surface_type == 'plane' and '$(arg plane_visual_mesh)' != ''}">
+      <visual name="photo_board">
+        <geometry><mesh filename="$(arg plane_visual_mesh)"/></geometry>
+      </visual>
+      <collision name="photo_board">
+        <origin xyz="0 0 ${-float('$(arg plane_size_m)'.split()[2])/2}"/>
+        <geometry><box size="$(arg plane_size_m)"/></geometry>
+      </collision>
+      </xacro:if>
+      <xacro:unless value="${surface_type == 'plane' and '$(arg plane_visual_mesh)' != ''}">
       <visual>
         <origin xyz="0 0 ${-0.0025 if surface_type == 'plane' else 0}"/>
@@ -34,4 +44,5 @@
       </collision>
       </xacro:unless>
+      </xacro:unless>
     </link>
     <joint name="jig_to_pen_surface" type="fixed"><parent link="pen_jig"/><child link="pen_surface"/><origin xyz="${surface_xyz}" rpy="${surface_rpy}"/></joint>
